File: HAM_Hat/HAM_Hat.kicad_sch (KiCad schematic)
At the start: 56 parts, among them J101 TL212V-02P-G12S, J102 DB-9RS-C, J103 NCW254-02S, J104 U.FL-R-SMT-1(80), J105 NCW200S-04R, J3 FHDH2.54-40, M101 Fan, Q101 BSS138, Q102 BSS138, Q103 BSS138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

Commit message: Add DCD LED
Parts:
- added D106: GRE, LED_SMD:LED_0603_1608Metric, symbol Device:LED
- added R114: 510R, Resistor_SMD:R_0603_1608Metric, symbol Device:R
Connections:
- net GND: now also D106.1 (K)
- net PTT: now also J3.32 (BCM12); no longer J3.11 (BCM17)
- net DCD: now reaches J3.36 (BCM16)
- net DCD: now also R114.1
- new net: D106.2 (A), R114.2
- no-connect marks 30 -> 28
Other:
- note added: "Carrier detect"

Commit message: LED moved
Parts:
- removed J104: U.FL-R-SMT-1(80), Connector_Coaxial:U.FL_Hirose_U.FL-R-SMT-1_Vertical, symbol Connector:Conn_Coaxial
- added J104: SMA6252A2, l_rf:SMA_angled, symbol default:levcsi_database/658
Connections:
- net GND: now also J104.2 (Ext)
- net at L102.2, U103.11 (RF_IN): now also J104.1 (In)
- no-connect marks 28 -> 29
Changed lines of the file:
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@@
 	)
 	(no_connect
+		(at 50.8 69.85)
+	)
+	(no_connect
 		(at 50.8 72.39)
 	)
@@
 	)
 	(symbol
-		(lib_id "Connector:Conn_Coaxial")
-		(at 276.86 60.96 0)
-		(unit 1)
-		(exclude_from_sim no)
-		(in_bom yes)
-		(on_board yes)
-		(dnp no)
-		(property "Reference" "J104"
-			(at 279.4 61.595 0)
-			(effects
-				(font
-					(size 1.27 1.27)
-				)
-				(justify left)
-			)
-		)
-		(property "Value" "U.FL-R-SMT-1(80)"
-			(at 279.4 63.9064 0)
-			(effects
-				(font
-					(size 1.27 1.27)
-				)
-				(justify left)
-			)
-		)
-		(property "Footprint" "Connector_Coaxial:U.FL_Hirose_U.FL-R-SMT-1_Vertical"
-			(at 276.86 60.96 0)
-			(effects
-				(font
-					(size 1.27 1.27)
-				)
-				(hide yes)
-			)
-		)
-		(property "Datasheet" "~"
-			(at 276.86 60.96 0)
-			(effects
-				(font
-					(size 1.27 1.27)
-				)
-				(hide yes)
-			)
-		)
-		(property "Description" "coaxial connector (BNC, SMA, SMB, SMC, Cinch/RCA, LEMO, ...)"
-			(at 276.86 60.96 0)
-			(effects
-				(font
-					(size 1.27 1.27)
-				)
-				(hide yes)
-			)
-		)
-		(property "id" "806"
-			(at 276.86 60.96 0)
-			(effects
-				(font
-					(size 1.27 1.27)
-				)
-				(hide yes)
-			)
-		)
-		(pin "1"
-		)
-		(pin "2"
-		)
-		(instances
-			(project "HAM_Hat"
-				(path "/d746ec70-4f38-4eaf-8576-334127e7f74a"
-					(reference "J104")
-					(unit 1)
-				)
-			)
-		)
-	)
-	(symbol
 		(lib_id "power:GND")
 		(at 276.86 68.58 0)
@@
 					(unit 1)
 				)
+			)
+		)
+	)
+	(symbol
+		(lib_id "default:levcsi_database/658")
+		(at 276.86 60.96 0)
+		(unit 1)
+		(exclude_from_sim no)
+		(in_bom yes)
+		(on_board yes)
+		(dnp no)
+		(fields_autoplaced yes)
+		(property "Reference" "J104"
+			(at 279.4 59.9831 0)
+			(effects
+				(font
+					(size 1.27 1.27)
+				)
+				(justify left)
+			)
+		)
+		(property "Value" "SMA6252A2"
+			(at 279.4 62.5231 0)
+			(effects
+				(font
+					(size 1.27 1.27)
+				)
+				(justify left)
+			)
+		)
+		(property "Footprint" "l_rf:SMA_angled"
+			(at 276.86 60.96 0)
+			(effects
+				(font
+					(size 1.27 1.27)
+				)
+				(hide yes)
+			)
+		)
+		(property "Datasheet" "~"
+			(at 276.86 60.96 0)
+			(effects
+				(font
+					(size 1.27 1.27)
+				)
+				(hide yes)
+			)
+		)
+		(property "Description" "coaxial connector (BNC, SMA, SMB, SMC, Cinch/RCA, LEMO, ...)"
+			(at 276.86 60.96 0)
+			(effects
+				(font
+					(size 1.27 1.27)
+				)
+				(hide yes)
+			)
+		)
+		(property "Value2" ""
+			(at 276.86 60.96 0)
+			(effects
+				(font
+					(size 1.27 1.27)
+				)
+				(hide yes)
+			)
+		)
+		(property "Value3" ""
+			(at 276.86 60.96 0)
+			(effects
+				(font
+					(size 1.27 1.27)
+				)
+				(hide yes)
+			)
+		)
+		(property "id" "658"
+			(at 276.86 60.96 0)
+			(effects
+				(font
+					(size 1.27 1.27)
+				)
+				(hide yes)
+			)
+		)
+		(pin "2"
+		)
+		(pin "1"
+		)
+		(instances
+			(project ""
+				(path "/d746ec70-4f38-4eaf-8576-334127e7f74a"
+					(reference "J104")
+					(unit 1)
+				)

Commit message: Add shutdown switch interface
Parts:
- added C107: 100n, Capacitor_SMD:C_0603_1608Metric, symbol Device:C
- added J106: Conn_01x02, Connector_Wire:SolderWire-0.5sqmm_1x02_P4.6mm_D0.9mm_OD2.1mm, symbol Connector_Generic:Conn_01x02
Connections:
- net GND: now also C107.2, J106.2 (Pin_2)
- net SHUTDOWN: now reaches J3.37 (BCM26)
- net SHUTDOWN: now also C107.1, J106.1 (Pin_1)
- no-connect marks 29 -> 28

Commit message: Add run LED
Parts:
- added D107: RED, LED_SMD:LED_0603_1608Metric, symbol default:levcsi_database/258
- added R115: 510R, Resistor_SMD:R_0603_1608Metric, symbol Device:R
Connections:
- net GND: now also D107.1 (K)
- net RUN_LED: now reaches J3.26 (BCM7)
- net RUN_LED: now also R115.1
- new net: D107.2 (A), R115.2
- no-connect marks 28 -> 27
Other:
- note added: "Running"
